File: expanded/gerassic_expanded_kicad_new.sch (KiCad schematic (older format))
At the start: 244 parts, among them J1 Gate In 1, J10 Gate Out 2, J11 Gate Out 6, J12 Gate Out 3, J13 Gate Out 7, J14 Decay Voltage CV In, J15 Decay Resistance CV In, J16 Pitch CV In, J2 Gate In 2, J3 Gate In 4, J4 Barrel_Jack, J5 Audio Out, J6 Gate Out 0, J7 Gate Out 4, J8 Gate Out 1, J9 Gate Out 5, Q1 BC547, Q10 BC547, Q11 BC547, Q12 BC557, Q13 BC557, Q14 BC547, Q15 BC547, Q16 BC557, Q17 BC547, Q18 BC547, Q19 BC547, Q2 BC547, Q20 BC547, Q21 BC547, Q22 MMBFJ111, Q3 BC547, Q4 BC547, Q5 BC547, Q6 BC547, Q7 BC547, Q8 BC547, Q9 BC547, SW1 SW_Push, SW2 SW_Push, SW3 SW_Push, SW4 SW_SP3T, SW5 SW_SP3T, SW6 SW_SPDT, U1 4028, U10 SSI2164 (PDIP), U11 LMC6484, U12 LMC6484, U13 LMC6484, U2 4077, U3 LM7809_TO220, U4 LMC6484, U5 LMC6484, U6 LMC6484, U7 LMC6484, U8 LMC6484, U9 4067

Commit message: update schematic
primarily maps symbols to footprints, corrects CD4067 symbol with local
copy, and a few other misc cleanups
Parts:
- removed U4: LMC6484, symbol Amplifier_Operational:LM358
- removed U6: LMC6484, symbol Amplifier_Operational:TL072
- C1, C9: footprint (none) -> Capacitor_SMD:C_Elec_8x10.2
- C10, C11, C12, C13, C17, C18, C19, C2, C20, C3, C4, C5, C6, C7, C8: footprint (none) -> Capacitor_SMD:C_0805_2012Metric_Pad1.18x1.45mm_HandSolder
- C14, C15, C16: footprint (none) -> Capacitor_THT:C_Disc_D5.0mm_W2.5mm_P5.00mm
- C21: footprint (none) -> Capacitor_SMD:CP_Elec_6.3x7.7
- D1, D12, D13, D2, D3, D4: footprint Diode_THT:D_DO-41_SOD81_P10.16mm_Horizontal -> Diode_SMD:D_SOD-123
- D10, D11, D14, D15, D16, D17, D5, D6, D7, D8, D9: footprint (none) -> LED_THT:LED_D3.0mm
- J1, J10, J11, J12, J13, J14, J15, J16, J2, J3, J5, J6, J7, J8, J9: footprint (none) -> gerassic:ENB_NEWCOMBOJACK_PANEL
- J4: footprint (none) -> Connector_BarrelJack:BarrelJack_CUI_PJ-102AH_Horizontal
- Q1, Q10, Q11, Q12, Q13, Q14, Q15, Q16, Q17, Q18, Q19, Q2, Q20, Q21, Q3, Q4, Q5, Q6, Q7, Q8, Q9: footprint Package_TO_SOT_THT:TO-92_Inline -> Package_TO_SOT_SMD:SOT-23
- R1, R10, R100, R101, R102, R103, R104, R105, R106, R107, R108, R109, R11, R110, R111, R112, R113, R114, R115, R12, R13, R14, R15, R16, R17, R18, R19, R2, R20, R21, R22, R23, R24, R25, R26, R27, R28, R29, R3, R30, R31, R32, R33, R34, R35, R36, R37, R38, R39, R4, R40, R41, R42, R43, R44, R45, R46, R47, R48, R49, R5, R50, R51, R52, R53, R54, R55, R56, R57, R58, R59, R6, R60, R61, R62, R63, R64, R65, R66, R67, R68, R69, R7, R70, R71, R72, R73, R74, R75, R76, R77, R78, R79, R8, R80, R81, R82, R83, R84, R85, R86, R87, R88, R89, R9, R90, R91, R92, R99: footprint (none) -> Resistor_SMD:R_0805_2012Metric_Pad1.20x1.40mm_HandSolder
- R116, R117, R118, R119, R93, R94, R95, R96, R97, R98: footprint (none) -> Resistor_THT:R_Axial_DIN0207_L6.3mm_D2.5mm_P7.62mm_Horizontal
- RV1, RV10, RV11, RV12, RV13, RV14, RV15, RV16, RV17, RV18, RV19, RV2, RV20, RV21, RV22, RV23, RV24, RV25, RV26, RV3, RV30, RV4, RV5, RV6, RV7, RV8, RV9: footprint (none) -> Potentiometer_THT:Potentiometer_Alpha_RD901F-40-00D_Single_Vertical
- RV27, RV28, RV29: footprint (none) -> Potentiometer_THT:Potentiometer_Bourns_3296W_Vertical
- SW1, SW2, SW3: footprint (none) -> gerassic:SW_TAIWAY_PB
- SW4, SW5: footprint (none) -> gerassic:SW_TAIWAY_SP3T
- SW6: footprint (none) -> gerassic:SW_TAIWAY_SPDT
- U1: footprint (none) -> Package_SO:SOIC-16_3.9x9.9mm_P1.27mm
- U10: footprint (none) -> Package_DIP:DIP-16_W7.62mm_Socket
- U2, U5, U7, U8: footprint (none) -> Package_SO:SOIC-14_3.9x8.7mm_P1.27mm
- U5: renamed from U11; footprint (none) -> Package_SO:SOIC-14_3.9x8.7mm_P1.27mm
- U7: renamed from U12; footprint (none) -> Package_SO:SOIC-14_3.9x8.7mm_P1.27mm
- U8: renamed from U13; footprint (none) -> Package_SO:SOIC-14_3.9x8.7mm_P1.27mm
- U9: footprint (none) -> Package_SO:SOIC-24W_7.5x15.4mm_P1.27mm; symbol 4xxx_IEEE:4067 -> gerassic:4067
Connections:
- net +9V: no longer C1.2, C11.2, C13.2, C17.2, C2.1, C3.1, C4.1, C8.2, C9.2, D1.2 (A), D13.2 (A), D2.2 (A), D3.2 (A), J1.S, J10.T, J11.T, J12.T, J13.T, J14.S, J15.S, J16.S, J2.S, J3.S, J4.2, J5.S, J6.T, J7.T, J8.T, J9.T, Q1.3 (E), Q10.3 (E), Q11.3 (E), Q14.3 (E), Q15.3 (E), Q17.3 (E), Q18.3 (E), Q19.3 (E), Q2.3 (E), Q20.3 (E), Q21.3 (E), Q3.3 (E), Q4.3 (E), Q5.3 (E), Q6.3 (E), Q7.3 (E), Q8.3 (E), Q9.3 (E), R22.2, R24.1, R25.2, R27.1, R28.2, R30.1, R34.1, R35.1, R41.1, R43.1, R44.1, R45.1, R46.1, R56.1, R57.1, R66.1, R67.1, R68.1, R94.2, R96.2, R98.2, RV1.1, RV11.1, RV19.1, RV2.1, RV21.1, RV23.1, RV25.1, RV3.1, RV4.3, RV5.1, RV7.1, RV9.1, SW1.1, SW2.1, SW3.1, SW4.1, U1.11 (D), U1.5 (S9), U1.8 (VSS), U1.9 (S8), U10.9 (V-), U2.12, U2.13, U2.7 (VSS), U3.2 (GND), U5.11 (V-), U7.11 (V-), U8.11 (V-), U9.12 (Vss), U9.15 (~E)
- net MIDO: now also R64.2
- net PitchMinus4: now also U9.19 (A12); no longer U9.14 (Q12)
- net PitchMinus5: now also U9.18 (A13); no longer U9.19 (A13)
- net PitchMinus6: now also U9.17 (A14); no longer U9.18 (A14)
- net PitchMinus7: now also U9.16 (A15); no longer U9.17 (A15)
- new net GND: C1.2, C11.2, C13.2, C17.2, C2.1, C3.1, C4.1, C8.2, C9.2, D1.2 (A), D13.2 (A), D2.2 (A), D3.2 (A), J1.S, J10.T, J11.T, J12.T, J13.T, J14.S, J15.S, J16.S, J2.S, J3.S, J4.2, J5.S, J6.T, J7.T, J8.T, J9.T, Q1.3 (E), Q10.3 (E), Q11.3 (E), Q14.3 (E), Q15.3 (E), Q17.3 (E), Q18.3 (E), Q19.3 (E), Q2.3 (E), Q20.3 (E), Q21.3 (E), Q3.3 (E), Q4.3 (E), Q5.3 (E), Q6.3 (E), Q7.3 (E), Q8.3 (E), Q9.3 (E), R22.2, R24.1, R25.2, R27.1, R28.2, R30.1, R34.1, R35.1, R41.1, R43.1, R44.1, R45.1, R46.1, R56.1, R57.1, R66.1, R67.1, R68.1, R94.2, R96.2, R98.2, RV1.1, RV11.1, RV19.1, RV2.1, RV21.1, RV23.1, RV25.1, RV3.1, RV4.3, RV5.1, RV7.1, RV9.1, SW1.1, SW2.1, SW3.1, SW4.1, U1.11 (D), U1.5 (S9), U1.8 (VSS), U1.9 (S8), U10.9 (V-), U2.12, U2.13, U2.7 (VSS), U3.2 (GND), U5.11 (V-), U7.11 (V-), U8.11 (V-), U9.12 (Vss), U9.15 (~E)
